Commit message: feat: sim bringup with scene initializer, ground collision, gripper fixes
- World simplified: ground plane + non-static target cube (3cm, URDF-spawned)
- scene_initializer_node: adds ground plane (2x2x0.05) and target cube to
  MoveIt planning scene
- Gripper: all mimic joints now in ros2_control with GazeboSystem mimic
  support — fingers no longer flop under gravity
- Fixed libexec discovery for ament_python (data_files entry)
- Cube size was a Gazebo rendering issue (inline SDF boxes ignored size);
  switched to URDF spawn path

File: src/ur3e_sim_bringup/urdf/ur3e_with_effector.urdf.xacro (robot description, xacro)
@@ -56,4 +56,39 @@
         <state_interface name="velocity"/>
       </joint>
+      <joint name="robotiq_85_right_knuckle_joint">
+        <param name="mimic">robotiq_85_left_knuckle_joint</param>
+        <param name="multiplier">-1</param>
+        <command_interface name="position"/>
+        <state_interface name="position"/>
+        <state_interface name="velocity"/>
+      </joint>
+      <joint name="robotiq_85_left_inner_knuckle_joint">
+        <param name="mimic">robotiq_85_left_knuckle_joint</param>
+        <param name="multiplier">1</param>
+        <command_interface name="position"/>
+        <state_interface name="position"/>
+        <state_interface name="velocity"/>
+      </joint>
+      <joint name="robotiq_85_right_inner_knuckle_joint">
+        <param name="mimic">robotiq_85_left_knuckle_joint</param>
+        <param name="multiplier">-1</param>
+        <command_interface name="position"/>
+        <state_interface name="position"/>
+        <state_interface name="velocity"/>
+      </joint>
+      <joint name="robotiq_85_left_finger_tip_joint">
+        <param name="mimic">robotiq_85_left_knuckle_joint</param>
+        <param name="multiplier">-1</param>
+        <command_interface name="position"/>
+        <state_interface name="position"/>
+        <state_interface name="velocity"/>
+      </joint>
+      <joint name="robotiq_85_right_finger_tip_joint">
+        <param name="mimic">robotiq_85_left_knuckle_joint</param>
+        <param name="multiplier">1</param>
+        <command_interface name="position"/>
+        <state_interface name="position"/>
+        <state_interface name="velocity"/>
+      </joint>
     </ros2_control>
   </xacro:if>
