Commit message: fix: collision safety, calibrated grip, and a physically real cube
Three defects reported from testing: the arm clipped the cube on approach, the
fingers closed straight through it, and the arm made unsafe self-colliding and
wrapped-around moves. Plus the cube did not behave like a physical object.

Collision safety and motion
- SRDF wrongly disabled 66 gripper-vs-arm pairs (every gripper link vs
  forearm_link tagged "Adjacent" though it is 4 joints away, and vs shoulder/
  upper_arm/base tagged "Never"). MoveIt was blind to the self-collisions.
- joint_limits.yaml had no position limits, so all six joints kept the URDF's
  +/-2*pi and the planner chose wrapped-around and elbow-flipped branches.
  Now +/-pi, with shoulder_lift capped at 0.
- The IK fallback retried with avoid_collisions=False and streamed the raw
  solution to the controller as a single trajectory point, with no path
  checking at all. Now avoidance stays on, the request is seeded from the
  current joint state, solutions moving a joint more than 2 rad are rejected,
  and the path is planned through MoveIt.
- Restored the controller's mid-trajectory tolerance (0.0 -> 0.5 rad).

Gripper closure
- GRIPPER_CLOSED was a hardcoded 0.70 rad: a 10.6 mm pad gap around a 60 mm
  cube, driving the fingers 24.7 mm into it. It is derived from the object
  width now, against a stroke table measured off the running model.
- GripperActionController's default 0.01 rad goal tolerance sits inside the
  knuckle's jitter band, so the action returned neither success nor stall and
  the cycle hung in GRASP_CLOSE for 320 s. Widened, allow_stalling enabled,
  and the orchestrator now has a watchdog on gripper goals.

Planning scene and straight-line motion
- The cube was never added to the planning scene, so every plan went through
  it. It is published on detection, attached to tool0 while carried, and
  removed on release - before the gripper opens, since putting it back with
  the fingers still around it left later plans starting in collision.
- Descents, lifts and the depart are Cartesian straight lines; a free plan
  between the same poses arcs sideways into the cube.

A physically real cube
- The grasp plugin held the cube kinematic and re-posed it every tick, so it
  ignored gravity, could not be moved in the GUI, and snapped to a hardcoded
  rest_z on release. Disabled by default (use_grasp_fix:=true restores it).
- Finger pads get real contact and friction; the pad-chain mimic joints run
  PID force control, since gazebo_ros2_control's position interface is a
  kinematic teleport that cannot stall on an object.
- Physics step 4 ms -> 1 ms, contact dead-band removed, cube lightened to
  0.08 kg with higher friction and stiffer contact.
- Perception intersected the cube's top-face sightline with the table plane,
  putting the estimate ~11 mm off and letting a pad shove the cube; it now
  intersects at the object's top.

Verified over 4 cycles before the physics change: 0 self-collisions, 0 invalid
plans, 0 IK fallbacks, 17 straight-line segments solved at 100%. The friction
grasp itself is real but not yet reliable - it lifts and carries the cube but
creeps out before the place target. Measurements and next steps in PROGRESS.md.

File: src/ur3e_sim_bringup/urdf/ur3e_with_effector.urdf.xacro (robot description, xacro)
@@ -8,5 +8,9 @@
   <xacro:arg name="use_grasp_plugins" default="true"/>
   <xacro:arg name="use_mimic_plugin" default="true"/>
-  <xacro:arg name="use_grasp_fix" default="true"/>
+  <!-- The grasp plugin held the target kinematically and teleported it each
+       tick, so it ignored gravity, could not be moved in the Gazebo GUI, and
+       snapped to the floor on release. The gripper grips by friction now, so
+       it is off by default. Set use_grasp_fix:=true to get the old behaviour. -->
+  <xacro:arg name="use_grasp_fix" default="false"/>
   <xacro:include filename="$(find ur_description)/urdf/ur_macro.xacro"/>
   <xacro:include filename="$(find robotiq_description)/urdf/ur_to_robotiq_adapter.urdf.xacro"/>
@@ -99,6 +103,10 @@
     </ros2_control>
     <xacro:if value="$(arg use_mimic_plugin)">
-    <!-- Couple the passive Robotiq finger joints to the driver knuckle with
-         PID force control so both fingers physically close on the object. -->
+    <!-- Couple the passive Robotiq finger joints to the driver knuckle.
+         The two contact pads hang off the inner-knuckle and finger-tip joints,
+         so those four run PID force control (usePID) and can stall against a
+         grasped object. gazebo_ros2_control drives the knuckle itself by
+         kinematic SetPosition, which cannot stall - a pad on that joint would
+         simply squeeze the object out instead of holding it. -->
     <gazebo>
       <plugin filename="libur3e_mimic_joint_plugin.so" name="mimic_right_knuckle">
@@ -113,6 +121,7 @@
         <mimicJoint>robotiq_85_left_inner_knuckle_joint</mimicJoint>
         <multiplier>1.0</multiplier>
-        <maxEffort>20.0</maxEffort>
-        <kp>15.0</kp><kd>0.5</kd>
+        <maxEffort>2.0</maxEffort>
+        <kp>6.0</kp><kd>0.05</kd>
+        <usePID>true</usePID>
       </plugin>
       <plugin filename="libur3e_mimic_joint_plugin.so" name="mimic_right_inner_knuckle">
@@ -120,6 +129,7 @@
         <mimicJoint>robotiq_85_right_inner_knuckle_joint</mimicJoint>
         <multiplier>-1.0</multiplier>
-        <maxEffort>20.0</maxEffort>
-        <kp>15.0</kp><kd>0.5</kd>
+        <maxEffort>2.0</maxEffort>
+        <kp>6.0</kp><kd>0.05</kd>
+        <usePID>true</usePID>
       </plugin>
       <plugin filename="libur3e_mimic_joint_plugin.so" name="mimic_left_finger_tip">
@@ -127,6 +137,7 @@
         <mimicJoint>robotiq_85_left_finger_tip_joint</mimicJoint>
         <multiplier>-1.0</multiplier>
-        <maxEffort>20.0</maxEffort>
-        <kp>15.0</kp><kd>0.5</kd>
+        <maxEffort>2.0</maxEffort>
+        <kp>6.0</kp><kd>0.05</kd>
+        <usePID>true</usePID>
       </plugin>
       <plugin filename="libur3e_mimic_joint_plugin.so" name="mimic_right_finger_tip">
@@ -134,6 +145,7 @@
         <mimicJoint>robotiq_85_right_finger_tip_joint</mimicJoint>
         <multiplier>1.0</multiplier>
-        <maxEffort>20.0</maxEffort>
-        <kp>15.0</kp><kd>0.5</kd>
+        <maxEffort>2.0</maxEffort>
+        <kp>6.0</kp><kd>0.05</kd>
+        <usePID>true</usePID>
       </plugin>
     </gazebo>
@@ -150,6 +162,10 @@
         <left_finger_link>robotiq_85_left_finger_tip_link</left_finger_link>
         <right_finger_link>robotiq_85_right_finger_tip_link</right_finger_link>
-        <attach_threshold>0.35</attach_threshold>
-        <detach_threshold>0.15</detach_threshold>
+        <!-- Thresholds must sit below the closing angle the orchestrator actually
+             commands. That angle is derived from the object width (a 0.06 m cube
+             closes the knuckle to ~0.27 rad, not the 0.70 rad it used to command),
+             so a 0.35 rad attach threshold would never latch. -->
+        <attach_threshold>0.20</attach_threshold>
+        <detach_threshold>0.08</detach_threshold>
         <grasp_radius>0.14</grasp_radius>
         <palm_offset_z>0.16</palm_offset_z>
@@ -176,6 +192,7 @@
        the independently-driven links overlap slightly and Gazebo's contact
        solver ejects them (pieces fly off). collide_bitmask 0x00 makes them
-       collide with nothing, which stops that; the grasp is plugin-managed so the
-       fingers need no physics contact. They still render and move visually. -->
+       collide with nothing, which stops that. They still render and move
+       visually. This applies to the intermediate linkage only - the two pads
+       that actually touch the object need real contact, see below. -->
   <xacro:macro name="finger_no_collision" params="link">
     <gazebo reference="${link}">
@@ -189,6 +206,21 @@
     </gazebo>
   </xacro:macro>
-  <xacro:finger_no_collision link="robotiq_85_left_finger_tip_link"/>
-  <xacro:finger_no_collision link="robotiq_85_right_finger_tip_link"/>
+  <!-- The two finger pads are the only links that should touch the object. They
+       carry the grip, so they get real contact and high friction. The knuckle is
+       position controlled to the object's own width, which makes the pads behave
+       as a rigid clamp - the object is squeezed between them and held by
+       friction, rather than being carried by a plugin. -->
+  <xacro:macro name="finger_pad_contact" params="link">
+    <gazebo reference="${link}">
+      <mu1>3.0</mu1>
+      <mu2>3.0</mu2>
+      <kp>1e6</kp>
+      <kd>1.0</kd>
+      <minDepth>0.0</minDepth>
+      <maxVel>0.01</maxVel>
+    </gazebo>
+  </xacro:macro>
+  <xacro:finger_pad_contact link="robotiq_85_left_finger_tip_link"/>
+  <xacro:finger_pad_contact link="robotiq_85_right_finger_tip_link"/>
   <xacro:finger_no_collision link="robotiq_85_left_inner_knuckle_link"/>
   <xacro:finger_no_collision link="robotiq_85_right_inner_knuckle_link"/>
