Commit message: feat: end effector nodes, pick-and-place orchestrator, camera orientation fix
- GripperStateNode: reads /joint_states → publishes /gripper/position + /gripper/state
- VacuumControllerNode: /vacuum/control service + /vacuum/active publisher (placeholder)
- PickPlaceOrchestrator: async state machine using MoveIt2 /move_action + gripper control
- MotionExecutor: move_to_joints/gripper_command via FollowJointTrajectory/GripperCommand
- Camera: pitch=0 (downward-looking via OGRE -Z convention), add setup.cfg for ament_python
- Perception: relaxed HSV orange thresholds [0-30,160-180] with wide saturation range
- Bringup: wire gripper_state_node, fix static TF to match world camera pose

File: src/ur3e_sim_bringup/urdf/target_cube.urdf (robot description, URDF)
Before this commit: robot target_cube, 1 links, 0 joints
Links:
- link base_link: geometry collision box size=0.06 0.06 0.06; visual box size=0.06 0.06 0.06

File: src/ur3e_sim_bringup/urdf/ur3e_with_effector.urdf.xacro (robot description, xacro)
@@ -8,5 +8,5 @@
   <xacro:include filename="$(find ur_description)/urdf/ur_macro.xacro"/>
   <xacro:include filename="$(find robotiq_description)/urdf/ur_to_robotiq_adapter.urdf.xacro"/>
-  <xacro:include filename="$(find robotiq_description)/urdf/robotiq_2f_85_macro.urdf.xacro"/>
+  <xacro:include filename="$(find ur3e_sim_bringup)/urdf/robotiq_2f_85_macro.urdf.xacro"/>
   <link name="world"/>
   <xacro:ur_robot
@@ -20,4 +20,5 @@
     sim_gazebo="$(arg sim_gazebo)"
     initial_positions="${xacro.load_yaml('$(arg initial_positions_file)')}"
+    generate_ros2_control_tag="false"
   >
     <origin xyz="0 0 0" rpy="0 0 0"/>
@@ -30,23 +31,56 @@
       </plugin>
     </gazebo>
-  </xacro:if>
-  <xacro:ur_to_robotiq
-    prefix=""
-    connected_to="tool0"
-    rotation="0"
-  />
-  <xacro:robotiq_gripper
-    name="gripper"
-    prefix=""
-    parent="gripper_mount_link"
-    include_ros2_control="false"
-  >
-    <origin xyz="0 0 0" rpy="0 0 0"/>
-  </xacro:robotiq_gripper>
-  <xacro:if value="$(arg sim_gazebo)">
-    <ros2_control name="Gripper" type="system">
+    <ros2_control name="CombinedHardware" type="system">
       <hardware>
         <plugin>gazebo_ros2_control/GazeboSystem</plugin>
       </hardware>
+      <joint name="shoulder_pan_joint">
+        <command_interface name="position"/>
+        <command_interface name="velocity"/>
+        <command_interface name="effort"/>
+        <state_interface name="position"/>
+        <state_interface name="velocity"/>
+        <state_interface name="effort"/>
+      </joint>
+      <joint name="shoulder_lift_joint">
+        <command_interface name="position"/>
+        <command_interface name="velocity"/>
+        <command_interface name="effort"/>
+        <state_interface name="position"/>
+        <state_interface name="velocity"/>
+        <state_interface name="effort"/>
+      </joint>
+      <joint name="elbow_joint">
+        <command_interface name="position"/>
+        <command_interface name="velocity"/>
+        <command_interface name="effort"/>
+        <state_interface name="position"/>
+        <state_interface name="velocity"/>
+        <state_interface name="effort"/>
+      </joint>
+      <joint name="wrist_1_joint">
+        <command_interface name="position"/>
+        <command_interface name="velocity"/>
+        <command_interface name="effort"/>
+        <state_interface name="position"/>
+        <state_interface name="velocity"/>
+        <state_interface name="effort"/>
+      </joint>
+      <joint name="wrist_2_joint">
+        <command_interface name="position"/>
+        <command_interface name="velocity"/>
+        <command_interface name="effort"/>
+        <state_interface name="position"/>
+        <state_interface name="velocity"/>
+        <state_interface name="effort"/>
+      </joint>
+      <joint name="wrist_3_joint">
+        <command_interface name="position"/>
+        <command_interface name="velocity"/>
+        <command_interface name="effort"/>
+        <state_interface name="position"/>
+        <state_interface name="velocity"/>
+        <state_interface name="effort"/>
+      </joint>
       <joint name="robotiq_85_left_knuckle_joint">
         <command_interface name="position"/>
@@ -93,3 +127,16 @@
     </ros2_control>
   </xacro:if>
+  <xacro:ur_to_robotiq
+    prefix=""
+    connected_to="tool0"
+    rotation="0"
+  />
+  <xacro:robotiq_gripper
+    name="gripper"
+    prefix=""
+    parent="gripper_mount_link"
+    include_ros2_control="false"
+  >
+    <origin xyz="0 0 0" rpy="0 0 0"/>
+  </xacro:robotiq_gripper>
 </robot>
